File: peripheral-board/peripheral-board.kicad_pcb (KiCad board)
At the start: 2 copper layers, 110 x 45 mm, 17 parts, among them J1 Power, J2 Arduino Ports, J3 4WD controller, J4 Head, J5 LED1, J6 LED2, M1 UsbToUartX2, Q1 IRLR8113, Q2 IRLR8113

Commit message: First pcb version
Parts:
- added JP1: Jumper, Wire_Connections_Bridges:WireConnection_0.80mmDrill, F.Cu at (148.5, 71.5)
- added JP2: Jumper, Wire_Connections_Bridges:WireConnection_0.80mmDrill, F.Cu at (185.5, 63.0)
- added JP3: Jumper, Wire_Connections_Bridges:WireConnection_0.80mmDrill, F.Cu at (162.0, 68.5)
- R7: value 10K -> 1K
- R8: value 1K -> 10K
- moved R3 14.9 mm to (131.5, 71.5), turned to 180 degrees
- moved R2 13.7 mm to (140.5, 62.5), turned to 180 degrees
- moved R4 13.7 mm to (140.5, 67.5), turned to 180 degrees
- moved R8 12.5 mm to (169.0, 68.0), turned to 0 degrees
- moved R1 12.1 mm to (131.5, 62.5), turned to 180 degrees
- moved J3 10.0 mm to (155.5, 74.5), turned to 270 degrees
- moved R7 4.61 mm to (166.5, 79.5), turned to 270 degrees
- moved Q1 3.81 mm to (176.0, 62.0)
- moved R5 3.81 mm to (164.0, 59.5)
- moved R6 3.81 mm to (164.0, 64.5)
- moved J1 3.16 mm to (112.0, 63.0)
- moved Q2 2.92 mm to (176.0, 75.0)
Connections:
- J1 pad 2: +7.4V -> +5V
- J1 pad 3: +5V -> +7.4V
- M1 pad 1: (no net) -> Net-(M1-Pad1)
- Q1 pad 2: Net-(J5-Pad1) -> Net-(JP2-Pad1)
- R3 pad 1: Net-(J2-Pad3) -> Net-(JP1-Pad2)
- R4 pad 2: Net-(J2-Pad3) -> Net-(JP1-Pad2)
- R7 pad 1: GND -> Net-(Q2-Pad1)
- R7 pad 2: Net-(J2-Pad2) -> Net-(JP3-Pad2)
- R8 pad 1: Net-(Q2-Pad1) -> Net-(J2-Pad2)
- R8 pad 2: Net-(J2-Pad2) -> GND
Routing:
- net +5V: track 0.00 -> 237.9 mm
- net GND: track 0.00 -> 203.1 mm
- net Net-(J6-Pad1): track 0.00 -> 29.8 mm
- net +7.4V: track 0.00 -> 29.4 mm
- net Net-(J4-Pad3): track 0.00 -> 26.1 mm
- net Net-(J3-Pad3): track 0.00 -> 25.6 mm
- net Net-(J2-Pad4): track 0.00 -> 24.7 mm
- net Net-(J2-Pad2): track 0.00 -> 24.1 mm
- net Net-(J3-Pad4): track 0.00 -> 21.2 mm
- net Net-(J3-Pad5): track 0.00 -> 17.0 mm
- net Net-(J4-Pad4): track 0.00 -> 14.7 mm
- net Net-(J5-Pad1): track 0.00 -> 13.7 mm
- net Net-(J2-Pad1): track 0.00 -> 13.4 mm
- net Net-(J2-Pad3): track 0.00 -> 12.7 mm
- net Net-(JP1-Pad2): track 0.00 -> 8.91 mm
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